Commit message: Fixed frame transform for the camera. Gazebo points the camera in the x direction, whereas ORB_SLAM (and everyone else) uses the z direction convention. Adjusted rviz to use the zx plane and created a new camera frame to export as the real frame

File: vs_gazebo/urdf/robot.urdf (robot description, URDF)
Before this commit: robot robot_model, 7 links, 6 joints
Links:
- added link sim_cam, mass 0.1; collision sphere radius=0.025; visual sphere radius=0.025
- link usb_cam: mass 0.1 -> None; geometry 
Joints:
- removed joint top_to_usb_cam
- added joint top_to_sim_cam: type fixed, parent top, child sim_cam, origin xyz=0.06 0 0.05 rpy=0 0 0, limit effort=100 velocity=100
- added joint usb_cam_sim_cam: type fixed, parent sim_cam, child usb_cam, origin xyz=0 0 0 rpy=-1.59 0 -1.57, limit effort=100 velocity=100
